File: plc/verision_14in_14out/plc_14in_14out.kicad_pcb (KiCad board)
At the start: 2 copper layers, 114 parts, among them J1 Screw_Terminal_01x02, J2 Screw_Terminal_01x06, J3 Screw_Terminal_01x09, J4 Screw_Terminal_01x05, J5 Screw_Terminal_01x05, K1 UMS05-1A80-75L, K2 UMS05-1A80-75L, K3 UMS05-1A80-75L, K4 UMS05-1A80-75L, K5 UMS05-1A80-75L, K6 UMS05-1A80-75L, K7 UMS05-1A80-75L, K8 UMS05-1A80-75L, SW1 SW_DIP_x01, SW2 SW_DIP_x01, SW3 SW_DIP_x01, U1 tlp127, U10 TLP127, U11 tlp127, U12 tlp127, U13 tlp127, U14 tlp127, U15 74HC14, U16 74HC14, U17 74HC14, U18 74HC245, U19 Teensy3.2, U2 tlp127, U20 74HC245, U21 ULN2803A, U22 74AHC125, U23 74AHC125, U3 tlp127, U4 tlp127, U5 tlp127, U6 tlp127, U7 tlp127, U8 tlp127, U9 TLP127

Commit message: Added the PWM output with IGBT, the ethernet port.
Parts:
- added C15: 10uF, Capacitor_SMD:C_0805_2012Metric_Pad1.18x1.45mm_HandSolder, F.Cu at (116.5, 111.4)
- added C16: 0.1uF, Capacitor_SMD:C_0603_1608Metric_Pad1.08x0.95mm_HandSolder, F.Cu at (85.3, 140.0)
- added C17: 18pF, Capacitor_SMD:C_0603_1608Metric, F.Cu at (127.5, 114.7)
- added C18: 18pF, Capacitor_SMD:C_0603_1608Metric, F.Cu at (127.5, 121.3)
- added C19: 0.1uF, Capacitor_SMD:C_0805_2012Metric_Pad1.18x1.45mm_HandSolder, F.Cu at (98.8, 124.3)
- added C20: 0.1uF, Capacitor_SMD:C_0805_2012Metric_Pad1.18x1.45mm_HandSolder, F.Cu at (92.7, 134.6)
- added C21: 220uF, Capacitor_SMD:CP_Elec_6.3x7.7, F.Cu at (85.0, 127.9)
- added C22: 0.1uF, Capacitor_SMD:C_0805_2012Metric, F.Cu at (85.4, 135.5)
- added D23: LED, LED_SMD:LED_1206_3216Metric_Castellated, F.Cu at (168.0, 78.0)
- added D24: LED, LED_SMD:LED_1206_3216Metric_Castellated, F.Cu at (167.9, 27.4)
- added D25: LED, LED_SMD:LED_1206_3216Metric_Castellated, F.Cu at (167.9, 37.3)
- added D26: LED, LED_SMD:LED_1206_3216Metric_Castellated, F.Cu at (168.0, 49.7)
- added D27: LED, LED_SMD:LED_1206_3216Metric_Castellated, F.Cu at (168.0, 58.9)
- added D28: LED, LED_SMD:LED_1206_3216Metric_Castellated, F.Cu at (168.0, 68.2)
- added J10: Screw_Terminal_01x06, Connector_PinSocket_2.54mm:PinSocket_1x06_P2.54mm_Vertical, F.Cu at (42.3, 145.4)
- added J11: Screw_Terminal_01x02, TerminalBlock_Altech:Altech_AK300_1x02_P5.00mm_45-Degree, F.Cu at (26.7, 117.7)
- added J6: RJ45_LED, Connector_RJ:RJ45_Hanrun_HR911105A, F.Cu at (106.4, 132.3)
- added J7: Screw_Terminal_01x06, TerminalBlock_Altech:Altech_AK300_1x06_P5.00mm_45-Degree, F.Cu at (212.2, 75.8)
- added J8: Screw_Terminal_01x05, TerminalBlock_Altech:Altech_AK300_1x05_P5.00mm_45-Degree, F.Cu at (212.2, 38.5)
- added J9: Screw_Terminal_01x06, Connector_PinSocket_2.54mm:PinSocket_1x06_P2.54mm_Vertical, F.Cu at (42.3, 124.3)
- added L1: 0.1uH, Inductor_SMD:L_0805_2012Metric_Pad1.15x1.40mm_HandSolder, F.Cu at (92.7, 129.5)
- added Q1: IRG4PF50W, Package_TO_SOT_SMD:TO-252-2, F.Cu at (193.4, 77.7)
- added Q2: IRG4PF50W, Package_TO_SOT_SMD:TO-252-2, F.Cu at (193.4, 68.5)
- added Q3: IRG4PF50W, Package_TO_SOT_SMD:TO-252-2, F.Cu at (193.4, 59.2)
- added Q4: IRG4PF50W, Package_TO_SOT_SMD:TO-252-2, F.Cu at (193.4, 49.7)
- added Q5: IRG4PF50W, Package_TO_SOT_SMD:TO-252-2, F.Cu at (193.8, 37.3)
- added Q6: IRG4PF50W, Package_TO_SOT_SMD:TO-252-2, F.Cu at (193.8, 27.9)
- added R40: 2.7k, Resistor_SMD:R_0603_1608Metric, F.Cu at (103.0, 118.2)
- added R41: 10K, Resistor_SMD:R_0603_1608Metric, F.Cu at (90.6, 122.4)
- added R42: 10K, Resistor_SMD:R_0603_1608Metric, F.Cu at (92.8, 122.4)
- added R43: 10K, Resistor_SMD:R_0603_1608Metric, F.Cu at (94.9, 122.4)
- added R44: 470, Resistor_SMD:R_0603_1608Metric, F.Cu at (99.1, 139.8)
- added R45: 470, Resistor_SMD:R_0603_1608Metric, F.Cu at (122.4, 139.7)
- added R46: 49.9, Resistor_SMD:R_0805_2012Metric_Pad1.20x1.40mm_HandSolder, F.Cu at (96.3, 130.9)
- added R47: 49.9, Resistor_SMD:R_0805_2012Metric_Pad1.20x1.40mm_HandSolder, F.Cu at (100.7, 118.5)
- added R48: 49.9, Resistor_SMD:R_0805_2012Metric_Pad1.20x1.40mm_HandSolder, F.Cu at (101.2, 130.7)
- added R49: 49.9, Resistor_SMD:R_0805_2012Metric_Pad1.20x1.40mm_HandSolder, F.Cu at (97.5, 118.5)
- added R50: 1.2k, Resistor_SMD:R_1206_3216Metric_Pad1.30x1.75mm_HandSolder, F.Cu at (150.9, 52.5)
- added R51: 1k, Resistor_SMD:R_0603_1608Metric, F.Cu at (163.2, 77.2)
- added R52: 390, Resistor_SMD:R_0603_1608Metric_Pad0.98x0.95mm_HandSolder, F.Cu at (167.9, 75.4)
- added R53: 1k, Resistor_SMD:R_0805_2012Metric_Pad1.20x1.40mm_HandSolder, F.Cu at (182.5, 75.4)
- added R54: 1k, Resistor_SMD:R_0805_2012Metric_Pad1.20x1.40mm_HandSolder, F.Cu at (185.8, 76.5)
- added R55: 10k, Resistor_SMD:R_0805_2012Metric_Pad1.20x1.40mm_HandSolder, F.Cu at (183.3, 79.0)
- added R56: 1k, Resistor_SMD:R_0603_1608Metric, F.Cu at (163.3, 26.7)
- added R57: 1k, Resistor_SMD:R_0603_1608Metric, F.Cu at (163.3, 36.5)
- added R58: 1k, Resistor_SMD:R_0603_1608Metric, F.Cu at (163.3, 49.0)
- added R59: 1k, Resistor_SMD:R_0603_1608Metric, F.Cu at (163.3, 58.2)
- added R60: 1k, Resistor_SMD:R_0603_1608Metric, F.Cu at (163.3, 67.3)
- added R61: 390, Resistor_SMD:R_0603_1608Metric_Pad0.98x0.95mm_HandSolder, F.Cu at (168.0, 24.9)
- added R62: 390, Resistor_SMD:R_0603_1608Metric_Pad0.98x0.95mm_HandSolder, F.Cu at (167.9, 34.8)
- added R63: 390, Resistor_SMD:R_0603_1608Metric_Pad0.98x0.95mm_HandSolder, F.Cu at (168.0, 47.1)
- added R64: 390, Resistor_SMD:R_0603_1608Metric_Pad0.98x0.95mm_HandSolder, F.Cu at (167.8, 56.4)
- added R65: 390, Resistor_SMD:R_0603_1608Metric_Pad0.98x0.95mm_HandSolder, F.Cu at (168.4, 65.7)
- added R66: 1k, Resistor_SMD:R_0805_2012Metric_Pad1.20x1.40mm_HandSolder, F.Cu at (182.4, 25.0)
- added R67: 1k, Resistor_SMD:R_0805_2012Metric_Pad1.20x1.40mm_HandSolder, F.Cu at (186.2, 27.2)
- added R68: 10k, Resistor_SMD:R_0805_2012Metric_Pad1.20x1.40mm_HandSolder, F.Cu at (183.3, 29.3)
- added R69: 1k, Resistor_SMD:R_0805_2012Metric_Pad1.20x1.40mm_HandSolder, F.Cu at (182.4, 34.8)
- added R70: 1k, Resistor_SMD:R_0805_2012Metric_Pad1.20x1.40mm_HandSolder, F.Cu at (185.7, 36.7)
- added R71: 10k, Resistor_SMD:R_0805_2012Metric_Pad1.20x1.40mm_HandSolder, F.Cu at (183.1, 38.9)
- added R72: 1k, Resistor_SMD:R_0805_2012Metric_Pad1.20x1.40mm_HandSolder, F.Cu at (182.2, 47.1)
- added R73: 1k, Resistor_SMD:R_0805_2012Metric_Pad1.20x1.40mm_HandSolder, F.Cu at (185.7, 48.9)
- added R74: 10k, Resistor_SMD:R_0805_2012Metric_Pad1.20x1.40mm_HandSolder, F.Cu at (183.0, 50.9)
- added R75: 1k, Resistor_SMD:R_0805_2012Metric_Pad1.20x1.40mm_HandSolder, F.Cu at (182.2, 56.1)
- added R76: 1k, Resistor_SMD:R_0805_2012Metric_Pad1.20x1.40mm_HandSolder, F.Cu at (185.8, 58.4)
- added R77: 10k, Resistor_SMD:R_0805_2012Metric_Pad1.20x1.40mm_HandSolder, F.Cu at (183.1, 60.5)
- added R78: 1k, Resistor_SMD:R_0805_2012Metric_Pad1.20x1.40mm_HandSolder, F.Cu at (182.5, 65.7)
- added R79: 1k, Resistor_SMD:R_0805_2012Metric_Pad1.20x1.40mm_HandSolder, F.Cu at (185.8, 66.8)
- added R80: 10k, Resistor_SMD:R_0805_2012Metric_Pad1.20x1.40mm_HandSolder, F.Cu at (183.3, 69.2)
- added SW4: SW_DIP_x01, Connector_PinHeader_2.54mm:PinHeader_1x02_P2.54mm_Vertical, F.Cu at (90.7, 24.9)
- added SW5: SW_DIP_x01, Connector_PinHeader_2.54mm:PinHeader_1x02_P2.54mm_Vertical, F.Cu at (149.6, 56.9)
- added U24: ENC28J60x-SS, Package_SO:SSOP-28_5.3x10.2mm_P0.65mm, F.Cu at (110.7, 121.0)
- added U25: LD1117S33TR_SOT223, Package_TO_SOT_SMD:SOT-223-3_TabPin2, F.Cu at (84.5, 118.2)
- added U26: 74AHCT125, Package_SO:SOIC-14_3.9x8.7mm_P1.27mm, F.Cu at (152.9, 67.4)
- added U27: 74AHCT125, Package_SO:SOIC-14_3.9x8.7mm_P1.27mm, F.Cu at (154.2, 43.1)
- added U28: TLP127, Package_SO:MFSOP6-4_4.4x3.6mm_P1.27mm, F.Cu at (176.0, 76.7)
- added U29: TLP127, Package_SO:MFSOP6-4_4.4x3.6mm_P1.27mm, F.Cu at (176.3, 26.2)
- added U30: TLP127, Package_SO:MFSOP6-4_4.4x3.6mm_P1.27mm, F.Cu at (176.1, 36.1)
- added U31: TLP127, Package_SO:MFSOP6-4_4.4x3.6mm_P1.27mm, F.Cu at (176.0, 48.4)
- added U32: TLP127, Package_SO:MFSOP6-4_4.4x3.6mm_P1.27mm, F.Cu at (176.0, 57.7)
- added U33: TLP127, Package_SO:MFSOP6-4_4.4x3.6mm_P1.27mm, F.Cu at (176.0, 66.9)
- added Y1: 25Mhz, Crystal:Crystal_HC49-4H_Vertical, F.Cu at (122.6, 115.7)
- U19: value Teensy3.2 -> Teensy3.5_All_Pins; footprint teensy:Teensy30_31_32_All_Pins -> teensy:Teensy35_36_All_Pins
- U22, U23: value 74AHC125 -> 74AHCT125
- moved J1 15.9 mm to (26.9, 136.9)
- moved U19 5.79 mm to (118.5, 51.8)
- moved SW3 2.41 mm to (135.4, 115.1)
Connections:
- U19 pad 10: D10 -> Net-(U19-Pad10)
- U19 pad 11: D11 -> Net-(U19-Pad11)
- U19 pad 12: D12 -> CS
- U19 pad 13: D13 -> MOSI
- U19 pad 14: D14 -> MISO
- U19 pad 15: D15 -> Net-(U19-Pad15)
- U19 pad 17: GND -> Net-(U19-Pad17)
- U19 pad 2: D2 -> Net-(U19-Pad2)
- U19 pad 3: D3 -> Net-(U19-Pad3)
- U19 pad 33: 5V -> Net-(U19-Pad33)
- U19 pad 4: D4 -> Net-(U19-Pad4)
- U19 pad 40: Net-(U19-Pad40) -> SCK
- U19 pad 5: D5 -> Net-(U19-Pad5)
- U19 pad 50: Net-(U19-Pad50) -> D23
- U19 pad 53: GND -> Net-(SW4-Pad1)
- U19 pad 6: D6 -> Net-(U19-Pad6)
- U19 pad 7: D7 -> Net-(U19-Pad7)
- U19 pad 8: D8 -> Net-(U19-Pad8)
- U19 pad 9: D9 -> Net-(U19-Pad9)
Routing:
- net 5V: track 314.9 -> 461.2 mm, vias 2 -> 4
- net CS: track 0.00 -> 98.3 mm, vias 0 -> 2
- net COM2: track 0.00 -> 86.3 mm, vias 0 -> 4
- net 3.3V: track 0.00 -> 78.6 mm, vias 0 -> 4
- net SCK: track 0.00 -> 78.5 mm, vias 0 -> 1
- net MOSI: track 0.00 -> 72.7 mm, vias 0 -> 1
- net MISO: track 0.00 -> 69.7 mm, vias 0 -> 1
- net Vge: track 0.00 -> 68.8 mm, vias 0 -> 4
- net OE1: track 0.00 -> 63.7 mm
- net +24V: track 0.00 -> 60.6 mm
- net 12V: track 0.00 -> 49.4 mm
- net RD+: track 0.00 -> 45.9 mm, vias 0 -> 1
- net Vge1: track 0.00 -> 44.7 mm, vias 0 -> 2
- net Net-(SW4-Pad1): track 0.00 -> 40.4 mm
- net COM4: track 0.00 -> 32.6 mm, vias 0 -> 1
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Other:
- board text added: "12V GND 24V"
- board text added: "5V GND 24V"
- board text added: "COM0 OUT0 OUT1 OUT2 OUT3"
- board text added: "COM1 OUT4 OUT5 OUT6 OUT7"
- board text added: "GND +24Vin"
- board text added: "GND 12Vout"
- board text added: "IN13 IN12 IN11 IN10 IN9 IN8"
- board text added: "IN7 IN6 IN5 IN4 IN3 IN2 IN1 IN0 1M"
- board text added: "OUT12 COM3 OUT13 COM4 Vge1"
- board text added: "OUT8 OUT9 OUT10 OUT11 COM2 VGE"
