File: plc/verision_14in_14out/plc_14in_14out.sch (KiCad schematic (older format))
At the start: 114 parts, among them J1 Screw_Terminal_01x02, J2 Screw_Terminal_01x06, J3 Screw_Terminal_01x09, J4 Screw_Terminal_01x05, J5 Screw_Terminal_01x05, K1 UMS05-1A80-75L, K2 UMS05-1A80-75L, K3 UMS05-1A80-75L, K4 UMS05-1A80-75L, K5 UMS05-1A80-75L, K6 UMS05-1A80-75L, K7 UMS05-1A80-75L, K8 UMS05-1A80-75L, SW1 SW_DIP_x01, SW2 SW_DIP_x01, SW3 SW_DIP_x01, U1 tlp127, U10 TLP127, U11 tlp127, U12 tlp127, U13 tlp127, U14 tlp127, U15 74HC14, U16 74HC14, U17 74HC14, U18 74HC245, U19 Teensy3.2, U2 tlp127, U20 74HC245, U21 ULN2803A, U22 74AHC125, U23 74AHC125, U3 tlp127, U4 tlp127, U5 tlp127, U6 tlp127, U7 tlp127, U8 tlp127, U9 TLP127

Commit message: Testing git.
This new version has a wire unconnected in the schematic.
Changed lines of the file:
@@
 Wire Wire Line
 	6900 9900 7050 9900
+Wire Wire Line
+	14650 5900 15300 5900
+Wire Wire Line
+	15300 5900 15300 6050
+Wire Wire Line
+	15300 6050 15000 6050
 $EndSCHEMATC

Commit message: Added the PWM output with IGBT, the ethernet port.
Parts:
- removed U19: Teensy3.2, teensy:Teensy30_31_32_All_Pins, symbol teensy:Teensy3.2
- added C15: 10uF, Capacitor_SMD:C_0805_2012Metric_Pad1.18x1.45mm_HandSolder, symbol Device:C
- added C16: 0.1uF, Capacitor_SMD:C_0603_1608Metric_Pad1.08x0.95mm_HandSolder, symbol Device:C
- added C17, C18: 18pF, Capacitor_SMD:C_0603_1608Metric, symbol Device:C
- added C19, C20: 0.1uF, Capacitor_SMD:C_0805_2012Metric_Pad1.18x1.45mm_HandSolder, symbol Device:C
- added C21: 220uF, Capacitor_SMD:CP_Elec_6.3x7.7, symbol Device:CP
- added C22: 0.1uF, Capacitor_SMD:C_0805_2012Metric, symbol Device:C
- added D23, D24, D25, D26, D27, D28: LED, LED_SMD:LED_1206_3216Metric_Castellated, symbol Device:LED
- added J10, J9: Screw_Terminal_01x06, Connector_PinSocket_2.54mm:PinSocket_1x06_P2.54mm_Vertical, symbol Connector:Screw_Terminal_01x06
- added J11: Screw_Terminal_01x02, TerminalBlock_Altech:Altech_AK300_1x02_P5.00mm_45-Degree, symbol Connector:Screw_Terminal_01x02
- added J6: RJ45_LED, Connector_RJ:RJ45_Hanrun_HR911105A, symbol Connector:RJ45_LED
- added J7: Screw_Terminal_01x06, TerminalBlock_Altech:Altech_AK300_1x06_P5.00mm_45-Degree, symbol Connector:Screw_Terminal_01x06
- added J8: Screw_Terminal_01x05, TerminalBlock_Altech:Altech_AK300_1x05_P5.00mm_45-Degree, symbol Connector:Screw_Terminal_01x05
- added L1: 0.1uH, Inductor_SMD:L_0805_2012Metric_Pad1.15x1.40mm_HandSolder, symbol pspice:INDUCTOR
- added Q1, Q2, Q3, Q4, Q5, Q6: IRG4PF50W, Package_TO_SOT_SMD:TO-252-2, symbol Transistor_IGBT:IRG4PF50W
- added R40: 2.7k, Resistor_SMD:R_0603_1608Metric, symbol Device:R
- added R41, R42, R43: 10K, Resistor_SMD:R_0603_1608Metric, symbol Device:R
- added R44, R45: 470, Resistor_SMD:R_0603_1608Metric, symbol Device:R
- added R46, R47, R48, R49: 49.9, Resistor_SMD:R_0805_2012Metric_Pad1.20x1.40mm_HandSolder, symbol Device:R
- added R50: 1.2k, Resistor_SMD:R_1206_3216Metric_Pad1.30x1.75mm_HandSolder, symbol Device:R
- added R51, R56, R57, R58, R59, R60: 1k, Resistor_SMD:R_0603_1608Metric, symbol Device:R
- added R52, R61, R62, R63, R64, R65: 390, Resistor_SMD:R_0603_1608Metric_Pad0.98x0.95mm_HandSolder, symbol Device:R
- added R53, R54, R66, R67, R69, R70, R72, R73, R75, R76, R78, R79: 1k, Resistor_SMD:R_0805_2012Metric_Pad1.20x1.40mm_HandSolder, symbol Device:R
- added R55, R68, R71, R74, R77, R80: 10k, Resistor_SMD:R_0805_2012Metric_Pad1.20x1.40mm_HandSolder, symbol Device:R
- added SW4, SW5: SW_DIP_x01, Connector_PinHeader_2.54mm:PinHeader_1x02_P2.54mm_Vertical, symbol Switch:SW_DIP_x01
- added U19: Teensy3.5_All_Pins, teensy:Teensy35_36_All_Pins, symbol teensy:Teensy3.5_All_Pins
- added U24: ENC28J60x-SS, Package_SO:SSOP-28_5.3x10.2mm_P0.65mm, symbol Interface_Ethernet:ENC28J60x-SS
- added U25: LD1117S33TR_SOT223, Package_TO_SOT_SMD:SOT-223-3_TabPin2, symbol Regulator_Linear:LD1117S33TR_SOT223
- added U26, U27: 74AHCT125, Package_SO:SOIC-14_3.9x8.7mm_P1.27mm, symbol 74AHC125:74AHC125
- added U28, U29, U30, U31, U32, U33: TLP127, Package_SO:MFSOP6-4_4.4x3.6mm_P1.27mm, symbol Isolator:TLP127
- added Y1: 25Mhz, Crystal:Crystal_HC49-4H_Vertical, symbol Device:Crystal
- U22, U23: value 74AHC125 -> 74AHCT125
Connections:
- net +24V: now also J10.5 (Pin_5), J10.6 (Pin_6), J9.5 (Pin_5), J9.6 (Pin_6)
- net 5V: now also J9.1 (Pin_1), J9.2 (Pin_2), R50.2, SW4.2, U25.3 (VI), U26.14 (VCC), U27.14 (VCC)
- net GND: now also C15.2, C16.2, C17.2, C18.2, C19.2, C20.2, C21.2, C22.2, D23.1 (K), D24.1 (K), D25.1 (K), D26.1 (K), D27.1 (K), D28.1 (K), J10.3 (Pin_3), J10.4 (Pin_4), J11.1 (Pin_1), J6.10, J6.11, J9.3 (Pin_3), J9.4 (Pin_4), R40.1, SW5.1, U19.1 (GND), U19.74 (GND), U24.11 (VSSRX), U24.18 (VSSTX), U24.2 (VSS), U24.21 (VSSPLL), U24.22 (VSSOSC), U25.1 (GND), U26.7 (GND), U27.7 (GND), U28.3, U29.3, U30.3, U31.3, U32.3, U33.3
- new net: C15.1, U24.1 (VCAP)
- new net: R40.2, U24.14 (RBIAS)
- new net: SW4.1, U19.53 (Vin)
- new net: R52.1, U28.1
- new net: J6.12, R45.2
- new net: J6.9, R44.1
- new net: D23.2 (A), R51.2
- new net: R53.2, U28.6
- new net: Q1.1 (G), R54.1
- new net: R54.2, R55.1, U28.4
- new net: C19.1, R47.2, R49.2
- new net: D28.2 (A), R60.2
- new net: R78.2, U33.6
- new net: R79.2, R80.1, U33.4
- new net: Q2.1 (G), R79.1
- new net: R65.1, U33.1
- new net: D27.2 (A), R59.2
- new net: R75.2, U32.6
- new net: R76.2, R77.1, U32.4
- new net: Q3.1 (G), R76.1
- new net: R64.1, U32.1
- new net: D26.2 (A), R58.2
- new net: R72.2, U31.6
- new net: R73.2, R74.1, U31.4
- new net: Q4.1 (G), R73.1
- new net: R63.1, U31.1
- new net: D25.2 (A), R57.2
- new net: R69.2, U30.6
- new net: R70.2, R71.1, U30.4
- new net: Q5.1 (G), R70.1
- new net: R62.1, U30.1
- new net: D24.2 (A), R56.2
- new net: R66.2, U29.6
- new net: R67.2, R68.1, U29.4
- new net: Q6.1 (G), R67.1
- new net: R61.1, U29.1
- new net 12V: J10.1 (Pin_1), J10.2 (Pin_2), J11.2 (Pin_2)
- new net 1Y1: R51.1, R52.2, U26.3 (1Y)
- new net 2Y1: R60.1, R65.2, U26.6 (2Y)
- new net 3.3V: C16.1, C21.1, C22.1, L1.1, R41.2, R42.2, R43.2, U24.15 (VDDTX), U24.19 (VDDRX), U24.20 (VDDPLL), U24.25 (VDDOSC), U24.28 (VDD), U25.2 (VO)
- new net 3Y1: R59.1, R64.2, U26.8 (3Y)
- new net 4Y1: R58.1, R63.2, U26.11 (4Y)
- new net 5Y1: U27.3 (1Y)
- new net 6Y1: U27.6 (2Y)
- new net 7Y1: R57.1, R62.2, U27.8 (3Y)
- new net 8Y1: R56.1, R61.2, U27.11 (4Y)
- new net CLKOUT: U24.3 (CLKOUT)
- new net COM2: J7.5 (Pin_5), Q1.3 (E), Q2.3 (E), Q3.3 (E), Q4.3 (E), R55.2, R74.2, R77.2, R80.2
- new net COM3: J8.2 (Pin_2), Q5.3 (E), R71.2
- new net COM4: J8.4 (Pin_4), Q6.3 (E), R68.2
- new net CS: R41.1, U19.12 (10_PWM_TX2_CS0), U24.9 (~CS)
- new net D23: U19.50 (23_A9_PWM_Touch), U27.12 (4A)
- new net INT: R42.1, U24.4 (~INT)
- new net LEDA: R44.2, U24.27 (LEDA)
- new net LEDB: R45.1, U24.26 (LEDB)
- new net MISO: U19.14 (12_MISO0), U24.6 (SO)
- new net MOSI: U19.13 (11_MOSI0), U24.7 (SI)
- new net O10: J7.3 (Pin_3), Q3.2 (C)
- new net O11: J7.4 (Pin_4), Q4.2 (C)
- new net O12: J8.1 (Pin_1), Q5.2 (C)
- new net O13: J8.3 (Pin_3), Q6.2 (C)
- new net O8: J7.1 (Pin_1), Q1.2 (C)
- new net O9: J7.2 (Pin_2), Q2.2 (C)
- new net OE1: R50.1, SW5.2, U26.1 (1OE), U26.10 (3OE), U26.13 (4OE), U26.4 (2OE), U27.1 (1OE), U27.10 (3OE), U27.13 (4OE), U27.4 (2OE)
- new net OSC1: C17.1, U24.23 (OSC1), Y1.1
- new net OSC2: C18.1, U24.24 (OSC2), Y1.2
- new net P4: C20.1, J6.4, L1.2, R46.1, R48.1
- new net RD+: J6.3, R47.1, U24.13 (TPIN+)
- new net RD-: J6.6, R49.1, U24.12 (TPIN-)
- new net RST: R43.1, U24.10 (~RESET)
- new net SCK: U19.40 (13_SCK0_LED), U24.8 (SCK)
- new net TD+: J6.1, R46.2, U24.17 (TPOUT+)
- new net TD-: J6.2, R48.2, U24.16 (TPOUT-)
- new net Vge: J7.6 (Pin_6), R53.1, R72.1, R75.1, R78.1
- new net Vge1: J8.5 (Pin_5), R66.1, R69.1
Other:
- note added: "DIGITALS OUTPUTS\n"
- note added: "INPUTS"
- note added: "Los ánodos de los leds son los pines 9 y 12, la imagen del led está mal en el componente\n"
- note added: "MODBUS COM\n"
- note added: "PWM OUTPUTS\n"
- moved on the sheet: D15, D16, D17, D18, D19, D20, D21, D22, J1, J4, J5, K1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
