File: plc/PackingMachineBoard/plc_14in_14out.sch (KiCad schematic (older format))
At the start: 195 parts, among them J1 Screw_Terminal_01x02, J10 Screw_Terminal_01x06, J11 Screw_Terminal_01x02, J2 Screw_Terminal_01x06, J3 Screw_Terminal_01x09, J4 Screw_Terminal_01x05, J5 Screw_Terminal_01x05, J6 RJ45_LED, J7 Screw_Terminal_01x06, J8 Screw_Terminal_01x05, J9 Screw_Terminal_01x06, K1 UMS05-1A80-75L, K2 UMS05-1A80-75L, K3 UMS05-1A80-75L, K4 UMS05-1A80-75L, K5 UMS05-1A80-75L, K6 UMS05-1A80-75L, K7 UMS05-1A80-75L, K8 UMS05-1A80-75L, Q1 IRG4PF50W, Q2 IRG4PF50W, Q3 IRG4PF50W, Q4 IRG4PF50W, Q5 IRG4PF50W, Q6 IRG4PF50W, SW1 SW_DIP_x01, SW2 SW_DIP_x01, SW3 SW_DIP_x01, SW4 SW_DIP_x01, SW5 SW_DIP_x01, U1 tlp127, U10 TLP127, U11 tlp127, U12 tlp127, U13 tlp127, U14 tlp127, U15 74HC14, U16 74HC14, U17 74HC14, U18 74HC245, U19 Teensy3.5_All_Pins, U2 tlp127, U20 74HC245, U21 ULN2803A, U22 74AHCT125, U23 74AHCT125, U24 ENC28J60x-SS, U25 LD1117S33TR_SOT223, U26 74AHCT125, U27 74AHCT125, U28 TLP127, U29 TLP127, U3 tlp127, U30 TLP127, U31 TLP127, U32 TLP127, U33 TLP127, U4 tlp127, U5 tlp127, U6 tlp127, U7 tlp127, U8 tlp127, U9 TLP127, Y1 25Mhz

Commit message: Version 1 lista con gerbers
Parts:
- removed J3: Screw_Terminal_01x09, TerminalBlock_Altech:Altech_AK300_1x09_P5.00mm_45-Degree, symbol Connector:Screw_Terminal_01x09
- removed J8: Screw_Terminal_01x05, TerminalBlock_Altech:Altech_AK300_1x05_P5.00mm_45-Degree, symbol Connector:Screw_Terminal_01x05
- added BT1: Battery_Cell, BatteryHolder_Keystone_103_1x20mm_new, symbol Device:Battery_Cell
- added C23, C24, C26: 0.1uF, Capacitor_SMD:C_1206_3216Metric, symbol Device:C
- added C25: 470uF, Capacitor_THT:C_Radial_D8.0mm_H11.5mm_P3.50mm, symbol Device:CP
- added C27: 220uF, Capacitor_SMD:CP_Elec_6.3x7.7, symbol Device:CP
- added D29: GREEN-LED, LED_SMD:LED_1206_3216Metric_Castellated, symbol Device:LED
- added D30: LED, LED_SMD:LED_1206_3216Metric_Castellated, symbol Device:LED
- added D31: D_Schottky, Diode_SMD:D_SMA_Handsoldering, symbol Device:D_Schottky
- added D32, D33: 1N47xxA, Diode_THT:D_DO-41_SOD81_P10.16mm_Horizontal, symbol Diode:1N47xxA
- added F1: Fuse, Fuse:Fuse_2920_7451Metric_Castellated, symbol Device:Fuse
- added J12: Ethernet, Connector_PinHeader_2.54mm:PinHeader_1x06_P2.54mm_Vertical, symbol Connector:Screw_Terminal_01x06
- added J13: Screw_Terminal_01x04, TerminalBlock_Altech:Altech_AK300_1x04_P5.00mm_45-Degree, symbol Connector:Screw_Terminal_01x04
- added J14: CAN, Connector_PinHeader_2.54mm:PinHeader_1x04_P2.54mm_Vertical, symbol Connector:Screw_Terminal_01x04
- added J15: SERIAL_1, Connector_PinHeader_2.54mm:PinHeader_1x04_P2.54mm_Vertical, symbol Connector:Screw_Terminal_01x04
- added J16: I2C0, Connector_PinHeader_2.54mm:PinHeader_1x04_P2.54mm_Vertical, symbol Connector:Screw_Terminal_01x04
- added J17: I2C1, Connector_PinHeader_2.54mm:PinHeader_1x04_P2.54mm_Vertical, symbol Connector:Screw_Terminal_01x04
- added J18, J20, J21, J22, J23, J24, J25: Screw_Terminal_01x01, Connector_PinHeader_2.54mm:PinHeader_1x01_P2.54mm_Vertical, symbol Connector:Screw_Terminal_01x01
- added J19: SERIAL_5, Connector_PinHeader_2.54mm:PinHeader_1x04_P2.54mm_Vertical, symbol Connector:Screw_Terminal_01x04
- added J3: Screw_Terminal_01x10, TerminalBlock_Altech:Altech_AK300_1x10_P5.00mm_45-Degree, symbol Connector:Screw_Terminal_01x10
- added J8: Screw_Terminal_01x06, TerminalBlock_Altech:Altech_AK300_1x06_P5.00mm_45-Degree, symbol Connector:Screw_Terminal_01x06
- added Q7: IRG4PF50W, Package_TO_SOT_SMD:TO-252-2, symbol Transistor_IGBT:IRG4PF50W
- added R81: 20k, Resistor_SMD:R_1206_3216Metric_Pad1.30x1.75mm_HandSolder, symbol Device:R
- added R82: 10K, Resistor_SMD:R_0603_1608Metric, symbol Device:R
- added R83: 1k, Resistor_SMD:R_0603_1608Metric, symbol Device:R
- added R84: 390, Resistor_SMD:R_0603_1608Metric_Pad0.98x0.95mm_HandSolder, symbol Device:R
- added R85, R86: 1k, Resistor_SMD:R_0805_2012Metric_Pad1.20x1.40mm_HandSolder, symbol Device:R
- added R87: 10k, Resistor_SMD:R_0805_2012Metric_Pad1.20x1.40mm_HandSolder, symbol Device:R
- added R88, R89, R91, R92: 10k, Resistor_SMD:R_1206_3216Metric, symbol Device:R
- added SW6: SW_DIP_x01, Button_Switch_THT:SW_DIP_SPSTx01_Slide_9.78x4.72mm_W7.62mm_P2.54mm, symbol Switch:SW_DIP_x01
- added unit 3 of U17
- added U34: tlp127, Package_SO:MFSOP6-4_4.4x3.6mm_P1.27mm, symbol Isolator:TLP127
- added U35: TLP127, Package_SO:MFSOP6-4_4.4x3.6mm_P1.27mm, symbol Isolator:TLP127
- added U36: LM7810_TO220, Package_TO_SOT_THT:TO-220-3_Vertical, symbol Regulator_Linear:LM7810_TO220
- SW4: value SW_DIP_x01 -> Prog
- U17: footprint (none) -> Package_SO:SOIC-14_3.9x8.7mm_P1.27mm
- U19: footprint teensy:Teensy35_36_All_Pins -> teensy:Teensy35_36_MODIFY
Connections:
- net labels added: 10V, A1, A2, A21, A22, AA14, AN2, AN3, CAN0Rx, CAN0Tx, D20, D21, D22, D24, D25, D26, D27, D28, D29, D30, D31, D32, D35, D36, D39, D43, D44, D45, D46, D47, D48, D49, D50, D55, D56, D57, IN14, O14, RX1, RX5, SCL0, SCL1, SDA0, SDA1, TX1, TX5, VBAT, Vin
- net labels removed: +24V, 6Y1, CLKOUT, D10, D11, D12, D13, D3, D4
- wire segments 310 -> 368
- no-connect marks 0 -> 34
Other:
- note added: "ANALOG INPUTS"
- note added: "Comunication"
- note added: "DIGITALS INPUTS"
- note added: "POWER SUPPLY"
- note removed: "INPUTS"
- moved on the sheet: J1, J10, J11, J2, J9, SW4

Commit message: Added a 3.3V and 5V pins Also commented the regulator used, and how to wire VGE and VGE1
Parts:
- added J26: 3V3, Connector_PinHeader_2.54mm:PinHeader_1x01_P2.54mm_Vertical, symbol Connector:Screw_Terminal_01x01
- added J27: 5V, Connector_PinHeader_2.54mm:PinHeader_1x01_P2.54mm_Vertical, symbol Connector:Screw_Terminal_01x01
- J10: value Screw_Terminal_01x06 -> DD2712SA - 12V
- J9: value Screw_Terminal_01x06 -> DD2712SA - 5V
Connections:
- net 3.3V: now also J26.1 (Pin_1)
- net 5V: now also J27.1 (Pin_1)
Other:
- note added: "Nota: A VGE y VGE1 se conectan los 12Vdc que entrega el regulador de voltage DD2712SA -12V"
Changed lines of the file:
@@
 P 2700 21200
 F 0 "J9" V 2664 20812 50  0000 R CNN
-F 1 "Screw_Terminal_01x06" V 2573 20812 50  0000 R CNN
+F 1 "DD2712SA - 5V" V 2573 20812 50  0000 R CNN
 F 2 "Connector_PinSocket_2.54mm:PinSocket_1x06_P2.54mm_Vertical" H 2700 21200 50  0001 C CNN
 F 3 "~" H 2700 21200 50  0001 C CNN
@@
 Wire Wire Line
 	2750 21400 2800 21400
-Wire Wire Line
-	2550 21450 2550 21400
 Connection ~ 2550 21400
 Wire Wire Line
@@
 P 2700 21900
 F 0 "J10" V 2664 21512 50  0000 R CNN
-F 1 "Screw_Terminal_01x06" V 2573 21512 50  0000 R CNN
+F 1 "DD2712SA - 12V" V 2573 21512 50  0000 R CNN
 F 2 "Connector_PinSocket_2.54mm:PinSocket_1x06_P2.54mm_Vertical" H 2700 21900 50  0001 C CNN
 F 3 "~" H 2700 21900 50  0001 C CNN
@@
 Text GLabel 1400 21900 2    50   Input ~ 0
 12V
-$Comp
-L teensy:Teensy3.5_All_Pins U19
-U 1 1 63E6F95E
-P 11900 14550
-F 0 "U19" H 11900 17293 60  0000 C CNN
-F 1 "Teensy3.5_All_Pins" H 11900 17187 60  0000 C CNN
-F 2 "teensy:Teensy35_36_MODIFY" H 11900 17081 60  0000 C CNN
-F 3 "https://www.pjrc.com/teensy/card8a_rev2.pdf" H 11900 38400 60  0001 C CNN
-F 4 "https://www.pjrc.com/teensy/pinout.html" H 10750 24550 50  0001 C CNN "Pinouts"
-	1    11900 14550
-	1    0    0    -1
-$EndComp
 Wire Wire Line
 	14250 15900 14200 15900
@@
 NoConn ~ 10950 1250
 NoConn ~ 11750 2300
-NoConn ~ 13050 13500
 NoConn ~ 13050 13000
 NoConn ~ 13050 12900
@@
 Wire Wire Line
 	900  21300 1100 21300
-Text GLabel 2550 21450 3    50   Input ~ 0
+Text GLabel 2550 21600 3    50   Input ~ 0
 5V
 Wire Wire Line
@@
 Wire Wire Line
 	3400 2450 3400 2800
+$Comp
+L teensy:Teensy3.5_All_Pins U19
+U 1 1 63E6F95E
+P 11900 14550
+F 0 "U19" H 11900 17293 60  0000 C CNN
+F 1 "Teensy3.5_All_Pins" H 11900 17187 60  0000 C CNN
+F 2 "teensy:Teensy35_36_MODIFY" H 11900 17081 60  0000 C CNN
+F 3 "https://www.pjrc.com/teensy/card8a_rev2.pdf" H 11900 38400 60  0001 C CNN
+F 4 "https://www.pjrc.com/teensy/pinout.html" H 10750 24550 50  0001 C CNN "Pinouts"
+	1    11900 14550
+	1    0    0    -1
+$EndComp
+$Comp
+L Connector:Screw_Terminal_01x01 J26
+U 1 1 637C4B7C
+P 14850 1750
+F 0 "J26" V 14814 1662 50  0000 R CNN
+F 1 "3V3" V 14723 1662 50  0000 R CNN
+F 2 "Connector_PinHeader_2.54mm:PinHeader_1x01_P2.54mm_Vertical" H 14850 1750 50  0001 C CNN
+F 3 "~" H 14850 1750 50  0001 C CNN
+	1    14850 1750
+	0    -1   -1   0
+$EndComp
+Wire Wire Line
+	13100 13500 13050 13500
+NoConn ~ 13100 13500
+Wire Wire Line
+	14850 1950 14850 2100
+$Comp
+L Connector:Screw_Terminal_01x01 J27
+U 1 1 6395B61D
+P 2200 21550
+F 0 "J27" H 2118 21325 50  0000 C CNN
+F 1 "5V" H 2118 21416 50  0000 C CNN
+F 2 "Connector_PinHeader_2.54mm:PinHeader_1x01_P2.54mm_Vertical" H 2200 21550 50  0001 C CNN
+F 3 "~" H 2200 21550 50  0001 C CNN
+	1    2200 21550
+	-1   0    0    1
+$EndComp
+Wire Wire Line
+	2550 21400 2550 21550
+Wire Wire Line
+	2400 21550 2550 21550
+Connection ~ 2550 21550
+Wire Wire Line
+	2550 21550 2550 21600
+Text Notes 20800 3350 0    79   ~ 0
+Nota: A VGE y VGE1 se conectan los 12Vdc que entrega el regulador de voltage DD2712SA -12V
 $EndSCHEMATC
